Commit message: M4: transport robot TRN-1 takes captured persons over
A slower transport UGV (trn1, 1.2 m/s, cargo box) parks east of the
detention building. The interceptor that captures a person holds him; the
nearest available transport is dispatched, stops next to him on the
detention side, takes him over (custody ESCORTING by TRN-1), escorts him
to the detention building and returns to its parking place. The
interceptor goes back to the defense at once. Without a transport, or if
it does not arrive within 90 s, the interceptor escorts him itself.

New roles DISPATCH, RETURN, STANDBY; transport variant of the robot
description and launch; transports argument (default trn1); the transport
is excluded from the detector like the other own robots, broadcasts its
position and is deconflicted. Unit tests for the pick-up point and the
choice of transport. README: TRN-1, quick start, open perception issue.

File: perimeter_defense_description/urdf/lup_ugv.urdf.xacro (robot description, xacro)
@@ -10,4 +10,6 @@
 <robot name="lup_ugv" xmlns:xacro="http://www.ros.org/wiki/xacro">
   <xacro:arg name="ns" default="lup1"/>
+  <!-- interceptor (LUP) or transport (TRN: same base with a cargo box, sand coloured) -->
+  <xacro:arg name="variant" default="interceptor"/>
   <xacro:arg name="enable_camera" default="true"/>
   <xacro:arg name="lidar_samples" default="720"/>
@@ -42,4 +44,5 @@
   <material name="black"><color rgba="0.08 0.08 0.08 1"/></material>
   <material name="grey"><color rgba="0.45 0.45 0.45 1"/></material>
+  <material name="sand"><color rgba="0.62 0.55 0.38 1"/></material>
   <xacro:macro name="box_inertia" params="m x y z">
     <inertia ixx="${m * (y*y + z*z) / 12.0}" ixy="0" ixz="0"
@@ -59,4 +62,12 @@
       <material name="olive"/>
     </visual>
+    <xacro:if value="${'$(arg variant)' == 'transport'}">
+      <visual>
+        <!-- Cargo box (visual only, below the lidar plane) -->
+        <origin xyz="-0.02 0 ${chassis_z_center + 0.19}"/>
+        <geometry><box size="0.40 0.32 0.24"/></geometry>
+        <material name="sand"/>
+      </visual>
+    </xacro:if>
     <collision>
       <origin xyz="0 0 ${chassis_z_center}"/>
